File: kicad/esp-prog-stick.kicad_sch (KiCad schematic)
At the start: 14 parts, among them J1 USB_A, J2 JST SM06B-SHLS-TF, Q1 S8050, Q2 S8050, U1 AZ1117-3.3, U2 CH340G, Y1 CSTNE12M0G550000R0

Commit message: Revision 2
Parts:
- removed C1: 10uF, Capacitor_SMD:C_0603_1608Metric, symbol Device:C
- removed C2: 22uF, Capacitor_SMD:C_1206_3216Metric_Pad1.33x1.80mm_HandSolder, symbol Device:C
- removed D1: DSL16, Diode_SMD:D_SOD-123F, symbol Device:D_Schottky
- removed D2: LED_Red, LED_SMD:LED_0603_1608Metric_Pad1.05x0.95mm_HandSolder, symbol Device:LED_Small
- removed J1: USB_A, USB_Custom:XKB_U217-041N, symbol Connector:USB_A
- removed J2: JST SM06B-SHLS-TF, Connector_JST:JST_SHL_SM06B-SHLS-TF_1x06-1MP_P1.00mm_Horizontal, symbol Connector:Conn_01x06_Socket
- removed Q1, Q2: S8050, Package_TO_SOT_SMD:SOT-23, symbol Transistor_BJT:S8050
- removed R1, R2: 10K, Resistor_SMD:R_0603_1608Metric, symbol Device:R
- removed R3: 2K2, Resistor_SMD:R_0603_1608Metric, symbol Device:R
- removed U1: AZ1117-3.3, Package_TO_SOT_SMD:SOT-223-3_TabPin2, symbol Regulator_Linear:AZ1117-3.3
- removed U2: CH340G, Package_SO:SOIC-16_3.9x9.9mm_P1.27mm, symbol Interface_USB:CH340G
- removed Y1: CSTNE12M0G550000R0, Crystal:Resonator_SMD_Murata_CSTxExxV-3Pin_3.0x1.1mm, symbol Device:Crystal_GND2_Small
Connections:
- no-connect marks 5 -> 0
Other:
- added sheet Board Outline (outline.kicad_sch)
- added sheet Layout (layout.kicad_sch)
- added sheet PCB Structure (pcb_structure.kicad_sch)
- added sheet Pinout (pinout.kicad_sch)
- added sheet Renders (renders.kicad_sch)
- added sheet Schematics (schematic.kicad_sch)
- added sheet Table of Contents (toc.kicad_sch)
- note added: "- Compatible with ESP8266 & ESP32 - CH340G USB-to-UART Bridge* - USB-A Plug - JST SHL Connector & replaceable Cable - 3.3V Power Supply - Power LED"
- note added: "ESP-PROG Stick"
- note added: "Features:"
- note removed: "3.3V Supply"
- note removed: "Auto Program"
- note removed: "PROG-Connector"
- note removed: "UART"
- note removed: "USB"
- company: github.com/harexew -> harexew.com // github.com/harexew
